Commit message: rviz + gz v02

File: robot_ws/src/openarm_description/assets/robot/openarm_v2.0/urdf/openarm_v20.urdf.xacro (robot description, xacro)
@@ -22,4 +22,7 @@
   <xacro:arg name="right_can_interface" default="can0" />
   <xacro:arg name="can_fd" default="true" />
+  <xacro:arg name="sim" default="none" />
+  <!-- Expose the arg as a property so expressions like ${sim == 'gz'} work. -->
+  <xacro:property name="sim" value="$(arg sim)" />
   <xacro:property name="robot_root" value="$(find openarm_description)/assets/robot/openarm_v2.0" />
   <xacro:property name="config_root" value="${robot_root + '/config'}" />
@@ -42,4 +45,5 @@
     right_can_interface="$(arg right_can_interface)"
     can_fd="$(arg can_fd)"
+    sim="$(arg sim)"
     ee_type="pinch_gripper"
     left_arm_prefix="left_"
@@ -47,3 +51,17 @@
     left_finger_mimic_multiplier="${pinch_finger_mimic_multiplier}"
     right_finger_mimic_multiplier="${pinch_finger_mimic_multiplier}" />
+  <!-- ========================= Gazebo (gz sim) ========================= -->
+  <!-- Only injected when launched with sim:=gz. Default sim:=none keeps the
+       robot_description identical for RViz / real hardware. -->
+  <xacro:if value="${sim == 'gz'}">
+    <gazebo>
+      <plugin filename="libgz_ros2_control-system.so"
+              name="gz_ros2_control::GazeboSimROS2ControlPlugin">
+        <parameters>$(find openarm_description)/config/gazebo/controllers.yaml</parameters>
+        <ros>
+          <namespace>/</namespace>
+        </ros>
+      </plugin>
+    </gazebo>
+  </xacro:if>
 </robot>

File: robot_ws/src/openarm_description/assets/robot/openarm_v2.0/urdf/ros2_control/openarm.bimanual.ros2_control.xacro (robot description, xacro)
@@ -25,14 +25,18 @@
              left_finger_mimic_multiplier:=^|1.0
              right_finger_mimic_multiplier:=^|1.0
-             can_fd:=^|true">
+             can_fd:=^|true
+             sim:=^|none">
     <ros2_control name="openarm_left_hardware_interface" type="system">
         <hardware>
           <param name="arm_type">${arm_type}</param>
-          <xacro:if value="${use_fake_hardware}">
+          <xacro:if value="${sim == 'gz'}">
+            <plugin>gz_ros2_control/GazeboSimSystem</plugin>
+          </xacro:if>
+          <xacro:if value="${use_fake_hardware and sim != 'gz'}">
             <plugin>mock_components/GenericSystem</plugin>
             <param name="fake_sensor_commands">${fake_sensor_commands}</param>
             <param name="state_following_offset">0.0</param>
           </xacro:if>
-          <xacro:unless value="${use_fake_hardware}">
+          <xacro:unless value="${use_fake_hardware or sim == 'gz'}">
             <plugin>openarm_hardware/OpenArmHW</plugin>
             <param name="can_interface">${left_can_interface}</param>
@@ -80,22 +84,28 @@
       <xacro:configure_joint joint_name="openarm_${left_arm_prefix}joint7" initial_position="0.0"/>
       <xacro:configure_joint joint_name="openarm_${left_arm_prefix}finger_joint1" initial_position="0.0" />
-      <!-- <joint name="openarm_${left_arm_prefix}finger_joint2">
-        <param name="mimic">openarm_${left_arm_prefix}finger_joint1</param>
-        <param name="multiplier">${left_finger_mimic_multiplier}</param>
-        <command_interface name="position"/>
+      <!-- Mimic finger: STATE INTERFACE ONLY.
+           gz_ros2_control refuses a command interface on a joint driven by
+           <mimic> in the URDF; the state interface is what makes
+           joint_state_broadcaster publish it (otherwise RViz complains about a
+           missing joint). Note: gz-sim physics does NOT enforce URDF <mimic>,
+           so finger_joint2 stays at 0 unless you also command it explicitly. -->
+      <joint name="openarm_${left_arm_prefix}finger_joint2">
         <state_interface name="position">
           <param name="initial_value">0.0</param>
         </state_interface>
-      </joint> -->
+      </joint>
     </ros2_control>
     <ros2_control name="openarm_right_hardware_interface" type="system">
         <hardware>
           <param name="arm_type">${arm_type}</param>
-          <xacro:if value="${use_fake_hardware}">
+          <xacro:if value="${sim == 'gz'}">
+            <plugin>gz_ros2_control/GazeboSimSystem</plugin>
+          </xacro:if>
+          <xacro:if value="${use_fake_hardware and sim != 'gz'}">
             <plugin>mock_components/GenericSystem</plugin>
             <param name="fake_sensor_commands">${fake_sensor_commands}</param>
             <param name="state_following_offset">0.0</param>
           </xacro:if>
-          <xacro:unless value="${use_fake_hardware}">
+          <xacro:unless value="${use_fake_hardware or sim == 'gz'}">
             <plugin>openarm_hardware/OpenArmHW</plugin>
             <param name="can_interface">${right_can_interface}</param>
@@ -127,12 +137,10 @@
       <xacro:configure_joint joint_name="openarm_${right_arm_prefix}joint7" initial_position="0.0"/>
       <xacro:configure_joint joint_name="openarm_${right_arm_prefix}finger_joint1" initial_position="0.0" />
-      <!-- <joint name="openarm_${right_arm_prefix}finger_joint2">
-        <param name="mimic">openarm_${right_arm_prefix}finger_joint1</param>
-        <param name="multiplier">${right_finger_mimic_multiplier}</param>
-        <command_interface name="position"/>
+      <!-- Mimic finger: STATE INTERFACE ONLY (see the left arm comment above). -->
+      <joint name="openarm_${right_arm_prefix}finger_joint2">
         <state_interface name="position">
           <param name="initial_value">0.0</param>
         </state_interface>
-      </joint> -->
+      </joint>
     </ros2_control>
   </xacro:macro>
