Commit message: v10 double arm with rviz gz2

File: robot_ws/src/openarm_description/assets/robot/openarm_v1.0/urdf/openarm_v10.urdf.xacro (robot description, xacro)
@@ -34,4 +34,7 @@
   <xacro:arg name="left_arm_base_rpy" default="-1.5708 0 0" />
   <xacro:arg name="can_fd" default="true" />
+  <xacro:arg name="sim" default="none" />
+  <!-- Expose the arg as a property so expressions like ${sim == 'gz'} work. -->
+  <xacro:property name="sim" value="$(arg sim)" />
   <xacro:property name="accepted_arm_types" value="${('v10', 'v1.0', 'v1_0', 'openarm_v10', 'openarm_v1.0', 'openarm_v1_0')}" />
   <xacro:if value="${'$(arg arm_type)' not in accepted_arm_types}">
@@ -80,4 +83,19 @@
   left_arm_base_rpy="$(arg left_arm_base_rpy)"
   can_fd="$(arg can_fd)"
+  sim="$(arg sim)"
   />
+  <!-- ========================= Gazebo (gz sim) ========================= -->
+  <!-- Only injected when launched with sim:=gz. Default sim:=none keeps the
+       robot_description identical for RViz / real hardware. -->
+  <xacro:if value="${sim == 'gz'}">
+    <gazebo>
+      <plugin filename="libgz_ros2_control-system.so"
+              name="gz_ros2_control::GazeboSimROS2ControlPlugin">
+        <parameters>$(find openarm_description)/config/gazebo/controllers.yaml</parameters>
+        <ros>
+          <namespace>/</namespace>
+        </ros>
+      </plugin>
+    </gazebo>
+  </xacro:if>
 </robot>

File: robot_ws/src/openarm_description/assets/robot/openarm_v1.0/urdf/robot/openarm_robot.xacro (robot description, xacro)
@@ -52,4 +52,5 @@
             right_arm_prefix:='right_'
             can_fd:='true'
+            sim:='none'
             "
             >
@@ -138,5 +139,6 @@
             right_arm_prefix="${right_arm_prefix}"
             hand="true"
-            ee_type="${ee_type}"/>
+            ee_type="${ee_type}"
+            sim="${sim}"/>
         </xacro:if>
     </xacro:if>
@@ -175,5 +177,6 @@
                 hand="true"
                 can_fd="${can_fd}"
-                ee_type="${ee_type}"/>
+                ee_type="${ee_type}"
+                sim="${sim}"/>
         </xacro:if>
     </xacro:if>

File: robot_ws/src/openarm_description/assets/robot/openarm_v1.0/urdf/ros2_control/openarm.bimanual.ros2_control.xacro (robot description, xacro)
@@ -24,15 +24,19 @@
              left_arm_prefix:=^|left_
              right_arm_prefix:=^|right_
-             can_fd:=^|true">
+             can_fd:=^|true
+             sim:=^|none">
     <!-- Left Arm Hardware Interface -->
     <ros2_control name="openarm_left_hardware_interface" type="system">
         <hardware>
           <param name="arm_type">${arm_type}</param>
-          <xacro:if value="${use_fake_hardware}">
+          <xacro:if value="${sim == 'gz'}">
+            <plugin>gz_ros2_control/GazeboSimSystem</plugin>
+          </xacro:if>
+          <xacro:if value="${use_fake_hardware and sim != 'gz'}">
             <plugin>mock_components/GenericSystem</plugin>
             <param name="fake_sensor_commands">${fake_sensor_commands}</param>
             <param name="state_following_offset">0.0</param>
           </xacro:if>
-          <xacro:unless value="${use_fake_hardware}">
+          <xacro:unless value="${use_fake_hardware or sim == 'gz'}">
             <plugin>openarm_hardware/OpenArmHW</plugin>
             <param name="can_interface">${left_can_interface}</param>
@@ -86,4 +90,15 @@
       <xacro:if value="${hand}">
         <xacro:configure_joint joint_name="openarm_${left_arm_prefix}finger_joint1" initial_position="0.0" />
+        <!-- Mimic finger: STATE INTERFACE ONLY.
+             gz_ros2_control refuses a command interface on a joint driven by
+             <mimic> in the URDF; the state interface is what makes
+             joint_state_broadcaster publish it (otherwise RViz complains about
+             a missing joint). gz-sim does keep the mimic constraint, so
+             finger_joint2 follows finger_joint1 in the simulation. -->
+        <joint name="openarm_${left_arm_prefix}finger_joint2">
+          <state_interface name="position">
+            <param name="initial_value">0.0</param>
+          </state_interface>
+        </joint>
       </xacro:if>
     </ros2_control>
@@ -92,10 +107,13 @@
         <hardware>
           <param name="arm_type">${arm_type}</param>
-          <xacro:if value="${use_fake_hardware}">
+          <xacro:if value="${sim == 'gz'}">
+            <plugin>gz_ros2_control/GazeboSimSystem</plugin>
+          </xacro:if>
+          <xacro:if value="${use_fake_hardware and sim != 'gz'}">
             <plugin>mock_components/GenericSystem</plugin>
             <param name="fake_sensor_commands">${fake_sensor_commands}</param>
             <param name="state_following_offset">0.0</param>
           </xacro:if>
-          <xacro:unless value="${use_fake_hardware}">
+          <xacro:unless value="${use_fake_hardware or sim == 'gz'}">
             <plugin>openarm_hardware/OpenArmHW</plugin>
             <param name="can_interface">${right_can_interface}</param>
@@ -133,4 +151,10 @@
       <xacro:if value="${hand}">
         <xacro:configure_joint joint_name="openarm_${right_arm_prefix}finger_joint1" initial_position="0.0" />
+        <!-- Mimic finger: STATE INTERFACE ONLY (see the left arm comment above). -->
+        <joint name="openarm_${right_arm_prefix}finger_joint2">
+          <state_interface name="position">
+            <param name="initial_value">0.0</param>
+          </state_interface>
+        </joint>
       </xacro:if>
     </ros2_control>

File: robot_ws/src/openarm_description/assets/robot/openarm_v1.0/urdf/ros2_control/openarm.ros2_control.xacro (robot description, xacro)
@@ -25,4 +25,5 @@
              bimanual:=false
              can_fd:=^|true
+             sim:=^|none
              no_prefix:=false">
     <xacro:property name="joint_prefix" value="${'' if no_prefix else 'openarm_' + arm_prefix}" />
@@ -31,10 +32,13 @@
           <param name="arm_type">${arm_type}</param>
           <param name="prefix">${arm_prefix}</param>
-          <xacro:if value="${use_fake_hardware}">
+          <xacro:if value="${sim == 'gz'}">
+            <plugin>gz_ros2_control/GazeboSimSystem</plugin>
+          </xacro:if>
+          <xacro:if value="${use_fake_hardware and sim != 'gz'}">
             <plugin>mock_components/GenericSystem</plugin>
             <param name="fake_sensor_commands">${fake_sensor_commands}</param>
             <param name="state_following_offset">0.0</param>
           </xacro:if>
-          <xacro:if value="${use_fake_hardware == 0}">
+          <xacro:if value="${use_fake_hardware == 0 and sim != 'gz'}">
             <plugin>openarm_hardware/OpenArmHW</plugin>
             <param name="can_interface">${can_interface}</param>
@@ -89,4 +93,10 @@
       <xacro:if value="${hand}">
         <xacro:configure_joint joint_name="${joint_prefix}finger_joint1" initial_position="0.0" />
+        <!-- Mimic finger: STATE INTERFACE ONLY (see the bimanual variant). -->
+        <joint name="${joint_prefix}finger_joint2">
+          <state_interface name="position">
+            <param name="initial_value">0.0</param>
+          </state_interface>
+        </joint>
       </xacro:if>
     </ros2_control>
